File: TESTTHINK.sch (EAGLE design)
At the start: 21 parts, among them J1 Digital_0_7, J2 Analog, J3 Digital_8_13

Commit message: Renamed files for project
Parts:
- removed SL1: Digital_0_7, freetronics:M08
- removed SL2: Analog, freetronics:M06SIP
- removed SL3: Digital_8_13, freetronics-original:M100.1
- removed SLP: Power, freetronics:M08
- R1, R2, R3: value 560R 0603 -> 560R
- R4: value 1K 0603 -> 1K
- R5: value 1K5 0603 -> 1K5
Connections:
- net 3V3: no longer SLP.4
- net 5V: no longer SLP.5
- net A0: no longer SL2.1
- net A1: no longer SL2.2
- net A2: no longer SL2.3
- net A3: no longer SL2.4
- net A4: no longer SL2.5
- net A5: no longer SL2.6
- net AREF: no longer SL3.8
- net D0_RX: no longer SL1.1
- net D10: no longer SL3.3
- net D11_MOSI: no longer SL3.4
- net D12_MISO: no longer SL3.5
- net D13_SCK: no longer SL3.6
- net D1_TX: no longer SL1.2
- net D2: no longer SL1.3
- net D3: no longer SL1.4
- net D4: no longer SL1.5
- net D5: no longer SL1.6
- net D6: no longer SL1.7
- net D7: no longer SL1.8
- net D8: no longer SL3.1
- net D9: no longer SL3.2
- net GND: no longer SL3.7, SLP.6, SLP.7
- net IOREF: no longer SLP.2
- net NC: no longer SLP.1
- net RESET: no longer SLP.3
- net SCL: no longer SL3.10
- net SDA: no longer SL3.9
- net VIN: no longer SLP.8
Other:
- note added: "Freetronics THINK Test Shield"
- note added: "SKU: TESTTHINK"
- note added: "V1.0 (2016-06-23)"
- note added: "tron.cc/testthink"
- note removed: "Freetronics I2C Test Shield"
- note removed: "SKU: TESTI2C"
- note removed: "V1.0 (2014-06-24)"
- note removed: "tron.cc/testi2c"
